File: usb2uart.kicad_pcb (KiCad board)
At the start: 2 copper layers, 16 parts, among them P1 CONN_5, P2 CONN_2, P3 CONN_2, P4 CONN_2, P5 CONN_10

Commit message: Add project files
Parts:
- C4: footprint Capacitors_ThroughHole:C_Radial_D5_L6_P2.5 -> Capacitors_ThroughHole:C_Rect_L7_W2.5_P5
- D1, D2: footprint LEDs:LED_1206 -> LEDs:LED-3MM
- moved R2 8.71 mm to (177.7, 109.8), turned to 0 degrees
- moved R3 8.68 mm to (177.7, 106.9), turned to 0 degrees
- moved D2 5.19 mm to (178.9, 104.1), turned to 180 degrees
- moved D1 5.01 mm to (178.8, 112.5), turned to 180 degrees
- moved C3 2.91 mm to (159.5, 112.0)
Connections:
- DD1 pad 15: (no net) -> Net-(DD1-Pad15)
- P5 pad 7: (no net) -> Net-(DD1-Pad15)
Routing:
- net Net-(D2-Pad2): track 0.00 -> 8.42 mm
- net Net-(DD1-Pad1): track 0.00 -> 7.97 mm
- net Net-(D1-Pad2): track 0.00 -> 6.96 mm
- net Net-(DD1-Pad22): track 0.00 -> 6.53 mm
- net Net-(DD1-Pad24): track 0.00 -> 6.50 mm
- net Net-(DD1-Pad23): track 0.00 -> 5.69 mm
Other:
- net class Default: clearance 0.5 -> 0.3
- rule trace_clearance: 0.5 -> 0.3

Commit message: Create board
Parts:
- added P6: CONN_4, Pin_Headers:Pin_Header_Straight_1x04, F.Cu at (163.1, 117.5)
- added P7: CONN_2, Pin_Headers:Pin_Header_Straight_1x02, F.Cu at (183.5, 117.5)
- added P8: CONN_1, Pin_Headers:Pin_Header_Straight_1x01, F.Cu at (170.0, 98.6)
- added REF**: R_0805, Resistors_SMD:R_0805, B.Cu at (159.5, 99.6)
- C3: footprint Capacitors_SMD:C_0805 -> Capacitors_ThroughHole:C_Rect_L7_W2.5_P5; moved to F.Cu
- D1, D2: moved to F.Cu
- P4: value CONN_2 -> CONN_1; footprint Pin_Headers:Pin_Header_Straight_1x02 -> Pin_Headers:Pin_Header_Straight_1x01
- P5: value CONN_10 -> CONN_4; footprint Pin_Headers:Pin_Header_Straight_1x10 -> Pin_Headers:Pin_Header_Straight_1x04
- R2, R3: footprint Resistors_SMD:R_0805 -> Resistors_ThroughHole:Resistor_Horizontal_RM10mm; moved to F.Cu
- moved P5 25.7 mm to (181.9, 98.6), turned to 270 degrees
- moved P3 20.4 mm to (175.8, 117.5), turned to 90 degrees
- moved P4 13.0 mm to (186.2, 98.6), turned to 0 degrees
- moved C3 11.1 mm to (167.6, 104.4)
- moved C1 10.7 mm to (185.2, 106.8)
- moved C4 7.84 mm to (170.2, 101.7), turned to 180 degrees
- moved R1 7.31 mm to (169.6, 104.4)
- moved DD1 4.02 mm to (172.8, 107.8), turned to 45 degrees
- moved P2 1.20 mm to (165.7, 98.6)
- moved R2 1.03 mm to (178.7, 109.6), turned to 180 degrees
- moved R3 1.03 mm to (178.7, 106.7), turned to 180 degrees
- moved DA1 0.87 mm to (152.9, 108.0), turned to 90 degrees
- moved D1 0.64 mm to (178.7, 111.9), turned to 0 degrees
- moved C2 0.60 mm to (165.6, 110.6)
- moved D2 0.33 mm to (178.7, 104.4), turned to 0 degrees
Connections:
- DA1 pad 2: Net-(C4-Pad1) -> Net-(DA1-Pad2)
- DA1 pad 4: Net-(DA1-Pad4) -> Net-(C4-Pad1)
- DD1 pad 10: (no net) -> Net-(DD1-Pad10)
- DD1 pad 3: Net-(DA1-Pad4) -> Net-(DA1-Pad3)
- DD1 pad 4: Net-(DA1-Pad3) -> Net-(DA1-Pad2)
- P1 pad 2: Net-(DA1-Pad3) -> Net-(DA1-Pad2)
- P1 pad 3: Net-(DA1-Pad4) -> Net-(DA1-Pad3)
- P4 pad 1: Net-(DD1-Pad11) -> Net-(DD1-Pad17)
- P5 pad 1: Net-(DD1-Pad1) -> Net-(DD1-Pad15)
- P5 pad 2: Net-(DD1-Pad24) -> Net-(DD1-Pad14)
- P5 pad 3: Net-(DD1-Pad23) -> Net-(DD1-Pad13)
- P5 pad 4: Net-(DD1-Pad22) -> Net-(DD1-Pad12)
Routing:
- net Net-(C1-Pad2): track 0.00 -> 119.8 mm
- net Net-(C4-Pad1): track 0.00 -> 65.8 mm
- net Net-(C1-Pad1): track 0.00 -> 30.5 mm
- net Net-(DA1-Pad2): track 0.00 -> 25.7 mm
- net Net-(DA1-Pad3): track 0.00 -> 23.1 mm
- net Net-(C2-Pad1): track 0.00 -> 20.1 mm
- net Net-(DA1-Pad1): track 0.00 -> 16.8 mm
- net Net-(D2-Pad2): track 8.42 -> 25.1 mm
- net Net-(DD1-Pad17): track 0.00 -> 16.2 mm
- net Net-(DD1-Pad15): track 0.00 -> 13.1 mm
- net Net-(DD1-Pad14): track 0.00 -> 11.1 mm
- net Net-(D1-Pad2): track 6.96 -> 17.6 mm
- net Net-(DD1-Pad20): track 0.00 -> 10.3 mm
- net Net-(DD1-Pad21): track 0.00 -> 9.00 mm
- net Net-(DD1-Pad13): track 0.00 -> 8.72 mm
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- added copper zone on B.Cu, net Net-(C1-Pad2)
Other:
- board outline added: 40.8 x 22.5 mm

Commit message: Fix board
Routing:
- net Net-(C1-Pad2): track 119.8 -> 118.6 mm
Other:
- board size 40.8 x 22.5 mm -> 39.7 x 22.5 mm
- net class Default: clearance 0.3 -> 0.4; trace_width 0.3 -> 0.4
- rule trace_clearance: 0.3 -> 0.4
Changed lines of the file:
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@@
     (links 43)
     (no_connects 1)
-    (area 147.117999 96.698999 188.035001 119.328001)
+    (area 141.605 91.821 190.563501 123.507501)
     (thickness 1.6)
     (drawings 9)
@@
   (page A4)
   (layers
-    (0 F.Cu signal)
+    (0 F.Cu signal hide)
     (31 B.Cu signal)
     (32 B.Adhes user)
@@
   )
   (setup
-    (last_trace_width 0.3)
-    (trace_clearance 0.3)
+    (last_trace_width 0.4)
+    (trace_clearance 0.4)
     (zone_clearance 0.508)
     (zone_45_only no)
@@
   (net 25 "Net-(DA1-Pad2)")
   (net_class Default "Это класс цепей по умолчанию."
-    (clearance 0.3)
-    (trace_width 0.3)
+    (clearance 0.4)
+    (trace_width 0.4)
     (via_dia 0.7)
     (via_drill 0.6)
@@
     )
   )
-  (gr_circle (center 149.098 98.552) (end 149.479 99.6315) (layer Edge.Cuts) (width 0.15))
-  (gr_circle (center 149.1615 117.4115) (end 149.5425 118.491) (layer Edge.Cuts) (width 0.15))
+  (gr_circle (center 150.241 98.679) (end 150.622 99.7585) (layer Edge.Cuts) (width 0.15))
+  (gr_circle (center 150.3045 117.2845) (end 150.6855 118.364) (layer Edge.Cuts) (width 0.15))
   (gr_circle (center 184.3405 102.743) (end 184.7215 103.8225) (layer Edge.Cuts) (width 0.15))
   (gr_circle (center 184.3405 113.792) (end 184.7215 114.8715) (layer Edge.Cuts) (width 0.15))
   (gr_line (start 187.96 119.253) (end 187.833 119.253) (angle 90) (layer Edge.Cuts) (width 0.15))
   (gr_line (start 187.96 96.774) (end 187.96 119.253) (angle 90) (layer Edge.Cuts) (width 0.15))
-  (gr_line (start 147.193 119.253) (end 187.833 119.253) (angle 90) (layer Edge.Cuts) (width 0.15))
-  (gr_line (start 147.193 96.774) (end 147.193 119.253) (angle 90) (layer Edge.Cuts) (width 0.15))
-  (gr_line (start 187.96 96.774) (end 147.193 96.774) (angle 90) (layer Edge.Cuts) (width 0.15))
+  (gr_line (start 148.27 119.253) (end 187.833 119.253) (angle 90) (layer Edge.Cuts) (width 0.15))
+  (gr_line (start 148.2725 96.774) (end 148.2725 119.253) (angle 90) (layer Edge.Cuts) (width 0.15))
+  (gr_line (start 187.96 96.774) (end 148.27 96.774) (angle 90) (layer Edge.Cuts) (width 0.15))
   (segment (start 185.166 106.807) (end 185.166 106.807) (width 0.3) (layer B.Cu) (net 1))
   (segment (start 175.387 105.649253) (end 174.389935 106.646318) (width 0.3) (layer B.Cu) (net 1))
@@
   (segment (start 157.734 111.76) (end 157.734 115.443) (width 0.3) (layer B.Cu) (net 2))
   (segment (start 157.734 115.443) (end 157.226 115.951) (width 0.3) (layer B.Cu) (net 2))
-  (segment (start 151.826 98.618) (end 159.512 98.618) (width 0.3) (layer B.Cu) (net 2))
+  (segment (start 152.5245 98.618) (end 159.512 98.618) (width 0.3) (layer B.Cu) (net 2))
   (segment (start 157.226 115.951) (end 155.956 117.221) (width 0.3) (layer B.Cu) (net 2))
   (segment (start 155.956 117.221) (end 152.4635 117.221) (width 0.3) (layer B.Cu) (net 2))
-  (segment (start 152.4635 117.221) (end 147.574 112.3315) (width 0.3) (layer B.Cu) (net 2))
-  (segment (start 147.574 112.3315) (end 147.574 102.87) (width 0.3) (layer B.Cu) (net 2))
-  (segment (start 147.574 102.87) (end 151.826 98.618) (width 0.3) (layer B.Cu) (net 2))
+  (segment (start 152.4635 117.221) (end 148.5265 113.284) (width 0.3) (layer B.Cu) (net 2))
+  (segment (start 148.5265 113.284) (end 148.5265 102.616) (width 0.3) (layer B.Cu) (net 2))
+  (segment (start 148.5265 102.616) (end 152.5245 98.618) (width 0.3) (layer B.Cu) (net 2))
   (segment (start 163.0826 110.6424) (end 163.0826 104.9001) (width 0.3) (layer B.Cu) (net 2))
   (segment (start 163.0826 104.9001) (end 162.5765 104.394) (width 0.3) (layer B.Cu) (net 2))
@@
   (segment (start 160.909 99.568) (end 161.4805 98.9965) (width 0.3) (layer B.Cu) (net 4))
   (segment (start 153.035 99.568) (end 160.909 99.568) (width 0.3) (layer B.Cu) (net 4))
-  (segment (start 148.9075 103.6955) (end 153.035 99.568) (width 0.3) (layer B.Cu) (net 4))
-  (segment (start 148.9075 112.0775) (end 148.9075 103.6955) (width 0.3) (layer B.Cu) (net 4))
-  (segment (start 153.035 116.205) (end 148.9075 112.0775) (width 0.3) (layer B.Cu) (net 4))
+  (segment (start 149.352 103.251) (end 153.035 99.568) (width 0.3) (layer B.Cu) (net 4))
+  (segment (start 149.352 112.522) (end 149.352 103.251) (width 0.3) (layer B.Cu) (net 4))
+  (segment (start 153.035 116.205) (end 149.352 112.522) (width 0.3) (layer B.Cu) (net 4))
   (segment (start 155.321 116.205) (end 153.035 116.205) (width 0.3) (layer B.Cu) (net 4))
   (segment (start 156.5275 114.9985) (end 155.321 116.205) (width 0.3) (layer B.Cu) (net 4))
@@
   (segment (start 178.816 106.8705) (end 178.6763 106.7308) (width 0.3) (layer B.Cu) (net 8))
   (segment (start 154.1526 101.95052) (end 153.06548 101.95052) (width 0.3) (layer B.Cu) (net 9))
-  (segment (start 153.06548 101.95052) (end 150.0505 104.9655) (width 0.3) (layer B.Cu) (net 9))
-  (segment (start 150.0505 104.9655) (end 150.0505 108.204) (width 0.3) (layer B.Cu) (net 9))
-  (segment (start 150.0505 108.204) (end 150.56612 108.71962) (width 0.3) (layer B.Cu) (net 9))
+  (segment (start 153.06548 101.95052) (end 150.241 104.775) (width 0.3) (layer B.Cu) (net 9))
+  (segment (start 150.241 104.775) (end 150.241 108.3945) (width 0.3) (layer B.Cu) (net 9))
+  (segment (start 150.241 108.3945) (end 150.56612 108.71962) (width 0.3) (layer B.Cu) (net 9))
   (segment (start 150.56612 108.71962) (end 151.80818 108.71962) (width 0.3) (layer B.Cu) (net 9))
   (segment (start 151.80818 108.71962) (end 151.80818 111.60506) (width 0.3) (layer B.Cu) (net 9))

Commit message: Add test board
Routing:
- net Net-(C1-Pad2): track 118.6 -> 96.6 mm
- net (no net): track 0.00 -> 3.87 mm
Other:
- net class Default: clearance 0.4 -> 0.3; trace_width 0.4 -> 0.3
- rule trace_clearance: 0.4 -> 0.3
