File: usb2uart.sch (KiCad schematic (older format))
At the start: 16 parts, among them P1 CONN_5, P2 CONN_2, P3 CONN_2, P4 CONN_2, P5 CONN_10

Commit message: Add project files
Parts:
- C4: footprint Capacitors_ThroughHole:C_Radial_D5_L6_P2.5 -> Capacitors_ThroughHole:C_Rect_L7_W2.5_P5
- D1, D2: footprint LEDs:LED_1206 -> LEDs:LED-3MM
Changed lines of the file:
@@
 LIBS:cp2110
 LIBS:sp0503baht
+LIBS:usb2uart-cache
 EELAYER 25 0
 EELAYER END
@@
 F 0 "C4" H 4500 4250 50  0000 L CNN
 F 1 "1.0" H 4500 4050 50  0000 L CNN
-F 2 "Capacitors_ThroughHole:C_Radial_D5_L6_P2.5" H 4450 4150 60  0001 C CNN
+F 2 "Capacitors_ThroughHole:C_Rect_L7_W2.5_P5" H 4450 4150 60  0001 C CNN
 F 3 "" H 4450 4150 60  0000 C CNN
 	1    4450 4150
@@
 F 0 "D1" H 6900 3050 50  0000 C CNN
 F 1 "LED" H 6900 2850 50  0000 C CNN
-F 2 "LEDs:LED_1206" H 6900 2950 60  0001 C CNN
+F 2 "LEDs:LED-3MM" H 6900 2950 60  0001 C CNN
 F 3 "" H 6900 2950 60  0000 C CNN
 	1    6900 2950
@@
 F 0 "D2" H 7200 3050 50  0000 C CNN
 F 1 "LED" H 7200 2850 50  0000 C CNN
-F 2 "LEDs:LED_1206" H 7200 2950 60  0001 C CNN
+F 2 "LEDs:LED-3MM" H 7200 2950 60  0001 C CNN
 F 3 "" H 7200 2950 60  0000 C CNN
 	1    7200 2950
@@
 	7200 3900 7700 3900
 Wire Wire Line
-	6400 3800 7100 3800
-Wire Wire Line
-	7100 3800 7100 4000
-Wire Wire Line
-	7100 4000 7700 4000
-Wire Wire Line
 	6400 3900 7000 3900
 Wire Wire Line
@@
 	3550 2700 3850 2700
 Connection ~ 3850 2700
+Wire Wire Line
+	7700 4000 7100 4000
+Wire Wire Line
+	7100 4000 7100 3800
+Wire Wire Line
+	7100 3800 6400 3800
 $EndSCHEMATC

Commit message: Create board
Parts:
- removed P4: CONN_2, Pin_Headers:Pin_Header_Straight_1x02, symbol CONN_2
- removed P5: CONN_10, Pin_Headers:Pin_Header_Straight_1x10, symbol CONN_10
- added P4, P8: CONN_1, Pin_Headers:Pin_Header_Straight_1x01, symbol CONN_1
- added P5, P6: CONN_4, Pin_Headers:Pin_Header_Straight_1x04, symbol CONN_4
- added P7: CONN_2, Pin_Headers:Pin_Header_Straight_1x02, symbol CONN_2
- C3: footprint Capacitors_SMD:C_0805 -> Capacitors_ThroughHole:C_Rect_L7_W2.5_P5
- DD1: symbol CP2110 -> CP2110-RESCUE-usb2uart
- R2, R3: footprint Resistors_SMD:R_0805 -> Resistors_ThroughHole:Resistor_Horizontal_RM10mm
Connections:
- wire segments 73 -> 75
Changed lines of the file:
@@
 EESchema Schematic File Version 2
+LIBS:usb2uart-rescue
 LIBS:power
 LIBS:device
@@
 $EndDescr
 $Comp
-L CP2110 DD1
+L CP2110-RESCUE-usb2uart DD1
 U 1 1 57FF75B0
 P 5550 3650
@@
 F 0 "C3" H 4200 4250 50  0000 L CNN
 F 1 "0.1" H 4200 4050 50  0000 L CNN
-F 2 "Capacitors_SMD:C_0805" H 4150 4150 60  0001 C CNN
+F 2 "Capacitors_ThroughHole:C_Rect_L7_W2.5_P5" H 4150 4150 60  0001 C CNN
 F 3 "" H 4150 4150 60  0000 C CNN
 	1    4150 4150
@@
 F 0 "R2" V 6980 2450 50  0000 C CNN
 F 1 "330" V 6900 2450 50  0000 C CNN
-F 2 "Resistors_SMD:R_0805" H 6900 2450 60  0001 C CNN
+F 2 "Resistors_ThroughHole:Resistor_Horizontal_RM10mm" H 6900 2450 60  0001 C CNN
 F 3 "" H 6900 2450 60  0000 C CNN
 	1    6900 2450
@@
 F 0 "R3" V 7280 2450 50  0000 C CNN
 F 1 "330" V 7200 2450 50  0000 C CNN
-F 2 "Resistors_SMD:R_0805" H 7200 2450 60  0001 C CNN
+F 2 "Resistors_ThroughHole:Resistor_Horizontal_RM10mm" H 7200 2450 60  0001 C CNN
 F 3 "" H 7200 2450 60  0000 C CNN
 	1    7200 2450
@@
 $EndComp
 $Comp
-L CONN_2 P4
-U 1 1 57FF9F41
-P 6600 4750
-F 0 "P4" V 6550 4750 40  0000 C CNN
-F 1 "CONN_2" V 6650 4750 40  0000 C CNN
-F 2 "Pin_Headers:Pin_Header_Straight_1x02" H 6600 4750 60  0001 C CNN
-F 3 "" H 6600 4750 60  0000 C CNN
-	1    6600 4750
-	0    1    1    0
-$EndComp
-$Comp
-L CONN_10 P5
-U 1 1 57FFA615
-P 8050 3850
-F 0 "P5" V 8000 3850 60  0000 C CNN
-F 1 "CONN_10" V 8100 3850 60  0000 C CNN
-F 2 "Pin_Headers:Pin_Header_Straight_1x10" H 8050 3850 60  0001 C CNN
-F 3 "" H 8050 3850 60  0000 C CNN
-	1    8050 3850
-	1    0    0    -1
-$EndComp
-$Comp
 L CONN_2 P2
 U 1 1 57FFB9C0
@@
 	0    1    -1   0
 $EndComp
-Wire Wire Line
-	2200 3100 4700 3100
-Wire Wire Line
-	2200 3200 4700 3200
-Wire Wire Line
-	2200 3300 3350 3300
-Wire Wire Line
-	3850 3700 4700 3700
-Wire Wire Line
-	4150 3500 4150 3950
-Wire Wire Line
-	3850 4400 3850 4350
-Wire Wire Line
-	3550 3950 3550 3400
-Wire Wire Line
-	3550 3400 4700 3400
-Wire Wire Line
-	3550 4350 3550 4400
-Connection ~ 3850 4400
-Wire Wire Line
-	4400 3300 4700 3300
-Wire Wire Line
-	3850 3300 3900 3300
-Wire Wire Line
-	2200 3000 4700 3000
-Wire Wire Line
-	4450 3000 4450 3950
-Wire Wire Line
-	4450 3600 4700 3600
-Connection ~ 4450 3600
-Connection ~ 4150 3700
-Wire Wire Line
-	4450 4400 4450 4350
-Wire Wire Line
-	3350 4400 4650 4400
-Wire Wire Line
-	4150 4350 4150 4400
-Connection ~ 4150 4400
-Wire Wire Line
-	3850 2150 3850 3950
-Wire Wire Line
-	4700 3500 4150 3500
-Connection ~ 3850 3700
-Connection ~ 4450 3000
-Wire Wire Line
-	6400 3500 7300 3500
-Wire Wire Line
-	6400 3700 7200 3700
-Connection ~ 3850 3300
-Wire Wire Line
-	6400 4300 6500 4300
-Wire Wire Line
-	6500 4300 6500 4400
-Wire Wire Line
-	6400 4200 6700 4200
-Wire Wire Line
-	6700 4200 6700 4400
-Wire Wire Line
-	6400 3000 6500 3000
-Wire Wire Line
-	6500 3000 6500 2900
-Wire Wire Line
-	6400 3100 6700 3100
-Wire Wire Line
-	6700 3100 6700 2900
-Wire Wire Line
-	7700 3500 7600 3500
-Wire Wire Line
-	7600 3500 7600 3200
-Wire Wire Line
-	7600 3200 6400 3200
-Wire Wire Line
-	7500 3600 7700 3600
-Wire Wire Line
-	7500 3600 7500 3300
-Wire Wire Line
-	7500 3300 6400 3300
-Wire Wire Line
-	7700 3400 6400 3400
-Wire Wire Line
-	6400 3600 7400 3600
-Wire Wire Line
-	7400 3600 7400 3700
-Wire Wire Line
-	7400 3700 7700 3700
-Wire Wire Line
-	7300 3500 7300 3800
-Wire Wire Line
-	7300 3800 7700 3800
-Wire Wire Line
-	7200 3150 7200 3900
-Wire Wire Line
-	7200 3900 7700 3900
-Wire Wire Line
-	6400 3900 7000 3900
-Wire Wire Line
-	7000 3900 7000 4100
-Wire Wire Line
-	7000 4100 7700 4100
-Wire Wire Line
-	6400 4000 6900 4000
-Wire Wire Line
-	6900 4000 6900 4200
-Wire Wire Line
-	6900 4200 7700 4200
-Wire Wire Line
-	6400 4100 6800 4100
-Wire Wire Line
-	6800 4100 6800 4300
-Wire Wire Line
-	6800 4300 7700 4300
-Wire Wire Line
-	6900 2700 6900 2750
-Wire Wire Line
-	7200 2700 7200 2750
-Wire Wire Line
-	6900 2200 6900 2150
-Wire Wire Line
-	3850 2150 7200 2150
-Wire Wire Line
-	7200 2150 7200 2200
-Wire Wire Line
-	6900 3150 6900 3500
-Connection ~ 6900 3500
-Connection ~ 7200 3700
-Connection ~ 6900 2150
-Wire Wire Line
-	3350 2600 3350 4400
-Connection ~ 3550 4400
-Wire Wire Line
-	4700 3800 4650 3800
-Wire Wire Line
-	4650 3800 4650 4400
-Connection ~ 4450 4400
-Connection ~ 3350 3300
-Wire Wire Line
-	2250 4400 2250 3400
-Wire Wire Line
-	2250 3400 2200 3400
 $Comp
 L CONN_5 P1
@@
 	-1   0    0    -1
 $EndComp
+$Comp
+L CONN_4 P5
+U 1 1 58048C85
+P 8100 4250
+F 0 "P5" V 8050 4250 50  0000 C CNN
+F 1 "CONN_4" V 8150 4250 50  0000 C CNN
+F 2 "Pin_Headers:Pin_Header_Straight_1x04" H 8100 4250 60  0001 C CNN
+F 3 "" H 8100 4250 60  0000 C CNN
+	1    8100 4250
+	1    0    0    -1
+$EndComp
+$Comp
+L CONN_4 P6
+U 1 1 5804AB2C
+P 8100 3550
+F 0 "P6" V 8050 3550 50  0000 C CNN
+F 1 "CONN_4" V 8150 3550 50  0000 C CNN
+F 2 "Pin_Headers:Pin_Header_Straight_1x04" H 8100 3550 60  0001 C CNN
+F 3 "" H 8100 3550 60  0000 C CNN
+	1    8100 3550
+	1    0    0    -1
+$EndComp
+$Comp
+L CONN_2 P7
+U 1 1 5804AB71
+P 8100 3900
+F 0 "P7" V 8050 3900 40  0000 C CNN
+F 1 "CONN_2" V 8150 3900 40  0000 C CNN
+F 2 "Pin_Headers:Pin_Header_Straight_1x02" H 8100 3900 60  0001 C CNN
+F 3 "" H 8100 3900 60  0000 C CNN
+	1    8100 3900
+	1    0    0    -1
+$EndComp
+$Comp
+L CONN_1 P8
+U 1 1 5804B757
+P 6700 4550
+F 0 "P8" H 6780 4550 40  0000 L CNN
+F 1 "CONN_1" H 6700 4605 30  0001 C CNN
+F 2 "Pin_Headers:Pin_Header_Straight_1x01" H 6700 4550 60  0001 C CNN
+F 3 "" H 6700 4550 60  0000 C CNN
+	1    6700 4550
+	0    1    1    0
+$EndComp
+$Comp
+L CONN_1 P4
+U 1 1 5804B7B0
+P 6500 4550
+F 0 "P4" H 6580 4550 40  0000 L CNN
+F 1 "CONN_1" H 6500 4605 30  0001 C CNN
+F 2 "Pin_Headers:Pin_Header_Straight_1x01" H 6500 4550 60  0001 C CNN
+F 3 "" H 6500 4550 60  0000 C CNN
+	1    6500 4550
+	0    1    1    0
+$EndComp
+Wire Wire Line
+	2200 3100 4700 3100
+Wire Wire Line
+	2200 3200 4700 3200
+Wire Wire Line
+	2200 3300 3350 3300
+Wire Wire Line
+	3850 3700 4700 3700
+Wire Wire Line
+	4150 3500 4150 3950
+Wire Wire Line
+	3850 4400 3850 4350
+Wire Wire Line
+	3550 3950 3550 3400
+Wire Wire Line
+	3550 3400 4700 3400
+Wire Wire Line
+	3550 4350 3550 4400
+Connection ~ 3850 4400
+Wire Wire Line
+	4400 3300 4700 3300
+Wire Wire Line
+	3850 3300 3900 3300
+Wire Wire Line
+	2200 3000 4700 3000
+Wire Wire Line
+	4450 3000 4450 3950
+Wire Wire Line
+	4450 3600 4700 3600
+Connection ~ 4450 3600
+Connection ~ 4150 3700
+Wire Wire Line
+	4450 4400 4450 4350
+Wire Wire Line
+	3350 4400 4650 4400
+Wire Wire Line
+	4150 4350 4150 4400
+Connection ~ 4150 4400
+Wire Wire Line
+	3850 2150 3850 3950
+Wire Wire Line
+	4700 3500 4150 3500
+Connection ~ 3850 3700
+Connection ~ 4450 3000
+Wire Wire Line
+	6400 3700 7200 3700
+Connection ~ 3850 3300
+Wire Wire Line
+	6400 4300 6500 4300
+Wire Wire Line
+	6500 4300 6500 4400
+Wire Wire Line
+	6400 4200 6700 4200
+Wire Wire Line
+	6700 4200 6700 4400
+Wire Wire Line
+	6400 3000 6500 3000
+Wire Wire Line
+	6500 3000 6500 2900
+Wire Wire Line
+	6400 3100 6700 3100
+Wire Wire Line
+	6700 3100 6700 2900
+Wire Wire Line
+	7400 3500 7400 3700
+Wire Wire Line
+	7400 3700 7750 3700
+Wire Wire Line
+	7300 3600 7300 3800
+Wire Wire Line
+	7300 3800 7750 3800
+Wire Wire Line
+	7200 3150 7200 4000
+Wire Wire Line
+	7200 4000 7750 4000
+Wire Wire Line
+	6400 3900 7000 3900
+Wire Wire Line
+	7000 3900 7000 4200
+Wire Wire Line
+	7000 4200 7750 4200
+Wire Wire Line
+	6400 4000 6900 4000
+Wire Wire Line
+	6900 4000 6900 4300
+Wire Wire Line
+	6900 4300 7750 4300
+Wire Wire Line
+	6400 4100 6800 4100
+Wire Wire Line
+	6800 4100 6800 4400
+Wire Wire Line
+	6800 4400 7750 4400
+Wire Wire Line
+	6900 2700 6900 2750
+Wire Wire Line
+	7200 2700 7200 2750
+Wire Wire Line
+	6900 2200 6900 2150
+Wire Wire Line
+	3850 2150 7200 2150
+Wire Wire Line
+	7200 2150 7200 2200
+Wire Wire Line
+	6900 3150 6900 3600
+Connection ~ 7200 3700
+Connection ~ 6900 2150
+Wire Wire Line
+	3350 2600 3350 4400
+Connection ~ 3550 4400
+Wire Wire Line
+	4700 3800 4650 3800
+Wire Wire Line
+	4650 3800 4650 4400
+Connection ~ 4450 4400
+Connection ~ 3350 3300
+Wire Wire Line
+	2250 4400 2250 3400
+Wire Wire Line
+	2250 3400 2200 3400
 Wire Wire Line
 	2250 4400 2500 4400
 Wire Wire Line
 	2500 4400 2500 4350
-Wire Wire Line
-	3000 3350 3000 3200
-Connection ~ 3000 3200
-Wire Wire Line
-	2750 3350 2750 3100
-Connection ~ 2750 3100
-Wire Wire Line
-	2500 3350 2500 3000
-Connection ~ 2500 3000
 Wire Wire Line
 	3550 2600 3550 2700
@@
 Connection ~ 3850 2700
 Wire Wire Line
-	7700 4000 7100 4000
-Wire Wire Line
-	7100 4000 7100 3800
+	7750 4100 7100 4100
+Wire Wire Line
+	7100 4100 7100 3800
 Wire Wire Line
 	7100 3800 6400 3800
+Wire Wire Line
+	6400 3600 7300 3600
+Connection ~ 6900 3600
+Wire Wire Line
+	7750 3400 7700 3400
+Wire Wire Line
+	7700 3400 7700 3200
+Wire Wire Line
+	7700 3200 6400 3200
+Wire Wire Line
+	7750 3500 7600 3500
+Wire Wire Line
+	7600 3500 7600 3300
+Wire Wire Line
+	7600 3300 6400 3300
+Wire Wire Line
+	7750 3600 7500 3600
+Wire Wire Line
+	7500 3600 7500 3400
+Wire Wire Line
+	7500 3400 6400 3400
+Wire Wire Line
+	7400 3500 6400 3500
+Wire Wire Line
+	3000 3350 3000 3000
+Connection ~ 3000 3000
+Wire Wire Line
+	2750 3350 2750 3200
+Connection ~ 2750 3200
+Wire Wire Line
+	2500 3350 2500 3100
+Connection ~ 2500 3100
 $EndSCHEMATC

Commit message: Refactoring
Parts:
- C1, C2, C4: symbol CP1 -> CP1-RESCUE-usb2uart
- C3: symbol C -> C-RESCUE-usb2uart
- D1, D2: symbol LED -> LED-RESCUE-usb2uart
- R1, R2, R3: symbol R -> R-RESCUE-usb2uart
Changed lines of the file:
@@
 LIBS:sp0503baht
 LIBS:usb2uart-cache
-EELAYER 25 0
+EELAYER 26 0
 EELAYER END
 $Descr A4 11693 8268
@@
 $EndComp
 $Comp
-L CP1 C4
+L CP1-RESCUE-usb2uart C4
 U 1 1 57FF80D7
 P 4450 4150
@@
 $EndComp
 $Comp
-L CP1 C2
+L CP1-RESCUE-usb2uart C2
 U 1 1 57FF83A0
 P 3850 4150
@@
 $EndComp
 $Comp
-L C C3
+L C-RESCUE-usb2uart C3
 U 1 1 57FF8439
 P 4150 4150
@@
 $EndComp
 $Comp
-L CP1 C1
+L CP1-RESCUE-usb2uart C1
 U 1 1 57FF8C97
 P 3550 4150
@@
 $EndComp
 $Comp
-L R R1
+L R-RESCUE-usb2uart R1
 U 1 1 57FF8D37
 P 4150 3300
@@
 $EndComp
 $Comp
-L LED D1
+L LED-RESCUE-usb2uart D1
 U 1 1 57FF9810
 P 6900 2950
@@
 $EndComp
 $Comp
-L LED D2
+L LED-RESCUE-usb2uart D2
 U 1 1 57FF9885
 P 7200 2950
@@
 $EndComp
 $Comp
-L R R2
+L R-RESCUE-usb2uart R2
 U 1 1 57FF98F0
 P 6900 2450
@@
 $EndComp
 $Comp
-L R R3
+L R-RESCUE-usb2uart R3
 U 1 1 57FF992F
 P 7200 2450
